Commit message: Added Hessian computation, and a bunch of testing

File: python/neural/examples/data/human_one_leg_inv.urdf (robot description, URDF)
Before this commit: robot jumper_inverted, 8 links, 7 joints
Links:
- added link world
Joints:
- added joint right_toe_root: type fixed, parent world, child right_toe
