Commit message: Enabled iLQR using cartesian loss

File: data/urdf/xmate3p/xmate3p.urdf (robot description, URDF)
Before this commit: robot xmate3, 9 links, 8 joints
Links:
- link xmate3_base: geometry visual mesh filename=meshes/visual/xmate3_base.stl scale=0.001 0.001 0.001
- link xmate3_link1: geometry visual mesh filename=meshes/visual/xmate3_link1.stl scale=0.001 0.001 0.001
- link xmate3_link2: geometry visual mesh filename=meshes/visual/xmate3_link2.stl scale=0.001 0.001 0.001
- link xmate3_link3: geometry visual mesh filename=meshes/visual/xmate3_link3.stl scale=0.001 0.001 0.001
- link xmate3_link4: geometry visual mesh filename=meshes/visual/xmate3_link4.stl scale=0.001 0.001 0.001
- link xmate3_link5: geometry visual mesh filename=meshes/visual/xmate3_link5.stl scale=0.001 0.001 0.001
- link xmate3_link6: geometry visual mesh filename=meshes/visual/xmate3_link6.stl scale=0.001 0.001 0.001
- link xmate3_link7: geometry visual mesh filename=meshes/visual/xmate3_link7.stl scale=0.001 0.001 0.001
Joints:
- joint joint1: axis 0 0 1 -> (none); limit lower=-3.0527 upper=3.0527 effort=300 velocity=10 -> (none); type revolute -> fixed
- joint joint2: axis 0 1 0 -> (none); limit lower=-2.0933 upper=2.0933 effort=300 velocity=10 -> (none); type revolute -> fixed
- joint joint5: axis 0 0 1 -> (none); limit lower=-3.0527 upper=3.0527 effort=300 velocity=10 -> (none); type revolute -> fixed
- joint joint7: axis 0 0 1 -> (none); limit lower=-6.283 upper=2.993 effort=300 velocity=10 -> (none); type revolute -> fixed
